Commit message: fix duplicate names

File: resources/anymal_c/urdf/anymal.urdf (robot description, URDF)
Before this commit: robot anymal, 78 links, 77 joints
Links:
- removed link LF_HAA
- removed link LF_HFE
- removed link LF_KFE
- removed link LH_HAA
- removed link LH_HFE
- removed link LH_KFE
- removed link RF_HAA
- removed link RF_HFE
- removed link RF_KFE
- removed link RH_HAA
- removed link RH_HFE
- removed link RH_KFE
- added link LF_HAA_link, mass 2.04; visual mesh filename=package://ocs2_robotic_assets/resources/anymal_c/meshes/dri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 scale=1.0 1.0 1.0
- added link LF_HFE_link, mass 2.04; collision cylinder length=0.14 radius=0.05; visual mesh filename=package://ocs2_robotic_assets/resources/anymal_c/meshes/dri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 scale=1.0 1.0 1.0
- added link LF_KFE_link, mass 2.04; collision cylinder length=0.14 radius=0.05; visual mesh filename=package://ocs2_robotic_assets/resources/anymal_c/meshes/dri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 scale=1.0 1.0 1.0
- added link LH_HAA_link, mass 2.04; visual mesh filename=package://ocs2_robotic_assets/resources/anymal_c/meshes/dri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 scale=1.0 1.0 1.0
- added link LH_HFE_link, mass 2.04; collision cylinder length=0.14 radius=0.05; visual mesh filename=package://ocs2_robotic_assets/resources/anymal_c/meshes/dri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 scale=1.0 1.0 1.0
- added link LH_KFE_link, mass 2.04; collision cylinder length=0.14 radius=0.05; visual mesh filename=package://ocs2_robotic_assets/resources/anymal_c/meshes/dri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 scale=1.0 1.0 1.0
- added link RF_HAA_link, mass 2.04; visual mesh filename=package://ocs2_robotic_assets/resources/anymal_c/meshes/dri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 scale=1.0 1.0 1.0
- added link RF_HFE_link, mass 2.04; collision cylinder length=0.14 radius=0.05; visual mesh filename=package://ocs2_robotic_assets/resources/anymal_c/meshes/dri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 scale=1.0 1.0 1.0
- added link RF_KFE_link, mass 2.04; collision cylinder length=0.14 radius=0.05; visual mesh filename=package://ocs2_robotic_assets/resources/anymal_c/meshes/dri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 scale=1.0 1.0 1.0
- added link RH_HAA_link, mass 2.04; visual mesh filename=package://ocs2_robotic_assets/resources/anymal_c/meshes/dri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 scale=1.0 1.0 1.0
- added link RH_HFE_link, mass 2.04; collision cylinder length=0.14 radius=0.05; visual mesh filename=package://ocs2_robotic_assets/resources/anymal_c/meshes/dri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 scale=1.0 1.0 1.0
- added link RH_KFE_link, mass 2.04; collision cylinder length=0.14 radius=0.05; visual mesh filename=package://ocs2_robotic_assets/resources/anymal_c/meshes/dri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 scale=1.0 1.0 1.0
Joints:
- joint LF_HAA: parent LF_HAA -> LF_HAA_link
- joint LF_HFE: parent LF_HFE -> LF_HFE_link
- joint LF_KFE: parent LF_KFE -> LF_KFE_link
- joint LF_hip_fixed_LF_HFE: child LF_HFE -> LF_HFE_link
- joint LF_thigh_fixed_LF_KFE: child LF_KFE -> LF_KFE_link
- joint LH_HAA: parent LH_HAA -> LH_HAA_link
- joint LH_HFE: parent LH_HFE -> LH_HFE_link
- joint LH_KFE: parent LH_KFE -> LH_KFE_link
- joint LH_hip_fixed_LH_HFE: child LH_HFE -> LH_HFE_link
- joint LH_thigh_fixed_LH_KFE: child LH_KFE -> LH_KFE_link
- joint RF_HAA: parent RF_HAA -> RF_HAA_link
- joint RF_HFE: parent RF_HFE -> RF_HFE_link
- joint RF_KFE: parent RF_KFE -> RF_KFE_link
- joint RF_hip_fixed_RF_HFE: child RF_HFE -> RF_HFE_link
- joint RF_thigh_fixed_RF_KFE: child RF_KFE -> RF_KFE_link
- joint RH_HAA: parent RH_HAA -> RH_HAA_link
- joint RH_HFE: parent RH_HFE -> RH_HFE_link
- joint RH_KFE: parent RH_KFE -> RH_KFE_link
- joint RH_hip_fixed_RH_HFE: child RH_HFE -> RH_HFE_link
- joint RH_thigh_fixed_RH_KFE: child RH_KFE -> RH_KFE_link
- joint base_LF_HAA: child LF_HAA -> LF_HAA_link
- joint base_LH_HAA: child LH_HAA -> LH_HAA_link
- joint base_RF_HAA: child RF_HAA -> RF_HAA_link
- joint base_RH_HAA: child RH_HAA -> RH_HAA_link
