Commit message: update franka inertial properties

File: resources/mobile_manipulator/franka/urdf/panda.urdf (robot description, URDF)
Before this commit: robot panda, 14 links, 13 joints
Links:
- removed link root
- link panda_hand: mass None -> 0.73
- link panda_leftfinger: mass None -> 0.1
- link panda_link0: mass None -> 2.0
- link panda_link1: mass None -> 4.970684
- link panda_link2: mass None -> 0.646926
- link panda_link3: mass None -> 3.228604
- link panda_link4: mass None -> 3.587895
- link panda_link5: mass None -> 1.225946
- link panda_link6: mass None -> 1.666555
- link panda_link7: mass None -> 7.35522e-01
- link panda_link8: mass None -> 0.01
- link panda_rightfinger: mass None -> 0.1
Joints:
- removed joint root_joint
- joint panda_finger_joint1: type prismatic -> fixed
- joint panda_finger_joint2: type prismatic -> fixed
