Commit message: update spot arm's inertial parameters to more reasonable values

File: resources/spot_arm/urdf/spot_arm.urdf (robot description, URDF)
Before this commit: robot spot_arm, 27 links, 26 joints
Links:
- link arm_link_el0: mass 0.725 -> 1.05
- link arm_link_el1: mass 0.725 -> 1.45
- link arm_link_fngr: mass 0.2 -> 0.25
- link arm_link_hr0: mass 1e-06 -> 1.0
- link arm_link_sh0: mass 2.3364000000000003 -> 1.594
- link arm_link_sh1: mass 0.2596 -> 1.0
- link arm_link_wr0: mass 0.98 -> 0.980
- link arm_link_wr1: mass 0.785 -> 0.535
Joints:
- joint arm_el1: limit lower=-2.79252680319092716487 upper=2.79252680319092716487 effort=30.3 velocity=10.0 -> lower=-2.79252680319092716487 upper=2.79252680319092716487 effort=90.9 velocity=10.0
- joint arm_f1x: axis 0.0 1.0 0.0 -> (none); limit lower=-1.57 upper=0.0 effort=15.32 velocity=10.0 -> (none); type revolute -> fixed
- joint arm_wr0: limit lower=-1.83259571459404613236 upper=1.83259571459404613236 effort=30.3 velocity=10.0 -> lower=-1.83259571459404613236 upper=1.83259571459404613236 effort=90.9 velocity=10.0
- joint arm_wr1: limit lower=-2.87979326579064354163 upper=2.87979326579064354163 effort=30.3 velocity=10.0 -> lower=-2.87979326579064354163 upper=2.87979326579064354163 effort=90.9 velocity=10.0
