Commit message: add d435 optical frame to g1 URDF

File: resources/g1/urdf/g1_29dof.urdf (robot description, URDF)
Before this commit: robot g1_29dof, 40 links, 39 joints
Links:
- added link d435_optical
Joints:
- added joint d435_optical_joint: type fixed, parent d435_link, child d435_optical, origin xyz=0 0 0 rpy=-1.5707963 0 -1.5707963
