Commit message: update spot inertial parameters for body and legs

File: resources/spot/urdf/spot.urdf (robot description, URDF)
Before this commit: robot spot, 30 links, 29 joints
Links:
- link base_inertia: mass 16.0 -> 32.86
- link fl_hip: mass 2.0 -> 1.68
- link fl_lleg: mass 0.5 -> 0.35
- link fl_uleg: mass 1.0 -> 2.34
- link fr_hip: mass 2.0 -> 1.68
- link fr_lleg: mass 0.5 -> 0.35
- link fr_uleg: mass 1.0 -> 2.34
- link hl_hip: mass 2.0 -> 1.68
- link hl_lleg: mass 0.5 -> 0.35
- link hl_uleg: mass 1.0 -> 2.34
- link hr_hip: mass 2.0 -> 1.68
- link hr_lleg: mass 0.5 -> 0.35
- link hr_uleg: mass 1.0 -> 2.34
